File: led-pwm-4bit.kicad_sch (KiCad schematic)
At the start: 38 parts, among them J1 24V IN, J2 LED STRIP, J3 HACKERBOARD, J4 FTDI-UPDI, Q1 RTR030N05HZG, U1 MCP1792T-3302H/CB, U2 ATtiny412-SSN

Commit message: Fuse the Hackerboard ground return and address review findings
Swapped J1 wires on a supply that shares ground with the printer put
supply + on board GND, which shorted through the Hackerboard ground.

- J3 pin 1 and J4 pins 1-2 move to a new net, HB_GND, which reaches
  board GND only through F2 (Bel 0ZCG0010FF2C, 0.1 A, 60 V, 100 A).
- R7-R10 rise to 10 kOhm to limit pin current while F2 is tripped.
- A DRC rule keeps copper 3.75 mm clear of the M3 mounting holes.
- The Mouser order rounds passives up to the 10-piece break with spares.
- Spec and README now cover source fusing, mounting, hot-plug
  overshoot, strip shorts and the remaining reverse-polarity limits.

Co-Authored-By: Claude Opus 5.5 <noreply@anthropic.com>
Parts:
- added F2: 0.1A 60V, Fuse:Fuse_1812_4532Metric, symbol Device:Polyfuse
- R10, R7, R8, R9: value 1k -> 10k; MPN RC0603FR-071KL -> RC0603FR-0710KL
Connections:
- net GND: now also F2.2; no longer J3.1 (Pin_1), J4.1 (Pin_1), J4.2 (Pin_2)
- new net HB_GND: F2.1, J3.1 (Pin_1), J4.1 (Pin_1), J4.2 (Pin_2)
