File: led-pwm-4bit.kicad_pcb (KiCad board)
At the start: 2 copper layers, 40 x 30 mm, 38 parts, among them J1 24V IN, J2 LED STRIP, J3 HACKERBOARD, J4 FTDI-UPDI, Q1 RTR030N05HZG, U1 MCP1792T-3302H/CB, U2 ATtiny412-SSN

Commit message: Fuse the Hackerboard ground return and address review findings
Swapped J1 wires on a supply that shares ground with the printer put
supply + on board GND, which shorted through the Hackerboard ground.

- J3 pin 1 and J4 pins 1-2 move to a new net, HB_GND, which reaches
  board GND only through F2 (Bel 0ZCG0010FF2C, 0.1 A, 60 V, 100 A).
- R7-R10 rise to 10 kOhm to limit pin current while F2 is tripped.
- A DRC rule keeps copper 3.75 mm clear of the M3 mounting holes.
- The Mouser order rounds passives up to the 10-piece break with spares.
- Spec and README now cover source fusing, mounting, hot-plug
  overshoot, strip shorts and the remaining reverse-polarity limits.

Co-Authored-By: Claude Opus 5.5 <noreply@anthropic.com>
Parts:
- added F2: 0.1A 60V, Fuse:Fuse_1812_4532Metric, F.Cu at (127.0, 102.2)
- R10, R7, R8, R9: value 1k -> 10k
Connections:
- J3 pad 1: GND -> /HB_GND
- J4 pad 1: GND -> /HB_GND
- J4 pad 2: GND -> /HB_GND
Changed lines of the file:
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@@
 		)
 	)
+	(footprint "Fuse:Fuse_1812_4532Metric"
+		(layer "F.Cu")
+		(at 127.05 102.15)
+		(descr "Fuse SMD 1812 (4532 Metric), square (rectangular) end terminal, IPC-7351 nominal, (Body size source: https://www.nikhef.nl/pub/departments/mt/projects/detectorR_D/dtddice/ERJ2G.pdf)")
+		(tags "fuse")
+		(property "Reference" "F2"
+			(at 0 0 0)
+			(layer "F.SilkS")
+			(effects
+				(font
+					(size 1 1)
+					(thickness 0.15)
+				)
+			)
+		)
+		(property "Value" "0.1A 60V"
+			(at 0 2.65 0)
+			(layer "F.Fab")
+			(effects
+				(font
+					(size 1 1)
+					(thickness 0.15)
+				)
+			)
+		)
+		(property "Datasheet" ""
+			(at 0 0 0)
+			(layer "F.Fab")
+			(hide yes)
+			(effects
+				(font
+					(size 1.27 1.27)
+				)
+			)
+		)
+		(property "Description" "PPTC in the Hackerboard and programmer ground return, 0.1 A hold, 60 V, 100 A"
+			(at 0 0 0)
+			(layer "F.Fab")
+			(hide yes)
+			(effects
+				(font
+					(size 1.27 1.27)
+				)
+			)
+		)
+		(property "KiLib_Generator" "SMD_2terminal_chip_molded"
+			(at 0 0 0)
+			(layer "F.SilkS")
+			(hide yes)
+			(effects
+				(font
+					(size 1 1)
+					(thickness 0.15)
+				)
+			)
+		)
+		(property "MPN" "0ZCG0010FF2C"
+			(at 0 0 0)
+			(layer "F.Fab")
+			(hide yes)
+			(effects
+				(font
+					(size 1.27 1.27)
+				)
+			)
+		)
+		(property "Manufacturer" "Bel Fuse"
+			(at 0 0 0)
+			(layer "F.Fab")
+			(hide yes)
+			(effects
+				(font
+					(size 1.27 1.27)
+				)
+			)
+		)
+		(sheetname "/")
+		(sheetfile "led-pwm-4bit.kicad_sch")
+		(attr smd)
+		(duplicate_pad_numbers_are_jumpers no)
+		(fp_line
+			(start -1.386252 -1.71)
+			(end 1.386252 -1.71)
+			(stroke
+				(width 0.15)
+				(type solid)
+			)
+			(layer "F.SilkS")
+		)
+		(fp_line
+			(start -1.386252 1.71)
+			(end 1.386252 1.71)
+			(stroke
+				(width 0.15)
+				(type solid)
+			)
+			(layer "F.SilkS")
+		)
+		(fp_rect
+			(start -2.95 -1.95)
+			(end 2.95 1.95)
+			(stroke
+				(width 0.05)
+				(type solid)
+			)
+			(fill no)
+			(layer "F.CrtYd")
+		)
+		(fp_rect
+			(start -2.25 -1.6)
+			(end 2.25 1.6)
+			(stroke
+				(width 0.1)
+				(type solid)
+			)
+			(fill no)
+			(layer "F.Fab")
+		)
+		(fp_text user "${REFERENCE}"
+			(at 0 0 0)
+			(layer "F.Fab")
+			(effects
+				(font
+					(size 1 1)
+					(thickness 0.15)
+				)
+			)
+		)
+		(pad "1" smd roundrect
+			(at -2.1375 0)
+			(size 1.125 3.4)
+			(layers "F.Cu" "F.Mask" "F.Paste")
+			(roundrect_rratio 0.222222)
+			(net "/HB_GND")
+		)
+		(pad "2" smd roundrect
+			(at 2.1375 0)
+			(size 1.125 3.4)
+			(layers "F.Cu" "F.Mask" "F.Paste")
+			(roundrect_rratio 0.222222)
+			(net "GND")
+		)
+		(embedded_fonts no)
+		(model "${KICAD10_3DMODEL_DIR}/Fuse.3dshapes/Fuse_1812_4532Metric.step"
+			(offset
+				(xyz 0 0 0)
+			)
+			(scale
+				(xyz 1 1 1)
+			)
+			(rotate
+				(xyz 0 0 0)
+			)
+		)
+	)
 	(footprint "Connector_PinHeader_2.54mm:PinHeader_1x06_P2.54mm_Vertical"
 		(locked yes)
@@
 		(tags "Through hole pin header THT 1x06 2.54mm single row")
 		(property "Reference" "J4"
-			(at 0 -2.464999 0)
+			(at 2 -0.4 0)
 			(layer "F.SilkS")
 			(effects
@@
 			(layers "*.Cu" "*.Mask")
 			(remove_unused_layers no)
-			(net "GND")
+			(net "/HB_GND")
 		)
 		(pad "2" thru_hole circle
@@
 			(layers "*.Cu" "*.Mask")
 			(remove_unused_layers no)
-			(net "GND")
+			(net "/HB_GND")
 		)
 		(pad "3" thru_hole circle
@@
 			)
 		)
-		(property "Value" "1k"
+		(property "Value" "10k"
 			(at 0 1.43 180)
 			(layer "F.Fab")
@@
 			)
 		)
-		(property "MPN" "RC0603FR-071KL"
+		(property "MPN" "RC0603FR-0710KL"
 			(at 0 0 180)
 			(layer "F.Fab")
@@
 			(layers "*.Cu" "*.Mask")
 			(remove_unused_layers no)
-			(net "GND")
+			(net "/HB_GND")
 		)
 		(pad "2" thru_hole circle
@@
 			)
 		)
-		(property "Value" "1k"
+		(property "Value" "10k"
 			(at 0 1.43 180)
 			(layer "F.Fab")
@@
 			)
 		)
-		(property "MPN" "RC0603FR-071KL"
+		(property "MPN" "RC0603FR-0710KL"
 			(at 0 0 180)
 			(layer "F.Fab")
@@
 		(tags "resistor")
 		(property "Reference" "R7"
-			(at 2 1.275001 0)
+			(at 2.25 0 0)
 			(layer "F.SilkS")
 			(effects
@@
 			)
 		)
-		(property "Value" "1k"
+		(property "Value" "10k"
 			(at 0 1.43 180)
 			(layer "F.Fab")
@@
 			)
 		)
-		(property "MPN" "RC0603FR-071KL"
+		(property "MPN" "RC0603FR-0710KL"
 			(at 0 0 180)
 			(layer "F.Fab")
@@
 		(tags "resistor")
 		(property "Reference" "R3"
-			(at 0 1.275001 0)
+			(at -2.05 0 90)
 			(layer "F.SilkS")
 			(effects
@@
 			)
 		)
-		(property "Value" "1k"
+		(property "Value" "10k"
 			(at 0 1.43 180)
 			(layer "F.Fab")
@@
 			)
 		)
-		(property "MPN" "RC0603FR-071KL"
+		(property "MPN" "RC0603FR-0710KL"
 			(at 0 0 180)
 			(layer "F.Fab")
@@
 				(font
 					(size 1.27 1.27)
+					(thickness 0.15)
 				)
 			)
@@
 				(font
 					(size 1.27 1.27)
+					(thickness 0.15)
 				)
 			)
@@
 		(layer "Edge.Cuts")
 	)
+	(gr_text "GND"
+		(at 135 102.4 0)
+		(layer "F.SilkS")
+		(effects
+			(font
+				(size 1 1)
+				(thickness 0.15)
+			)
+			(justify left)
+		)
+	)
 	(gr_text "24V IN"
 		(at 104.6 117.95 0)
@@
 		)
 	)
-	(gr_text "GND"
-		(at 131.85 102.399999 0)
-		(layer "F.SilkS")
-		(effects
-			(font
-				(size 1 1)
-				(thickness 0.15)
-			)
-			(justify right)
-		)
-	)

Commit message: pcb: Stitch the GND pours and give C6 a solid ground
Add 32 tented 0.6/0.3 mm GND vias: one beside each GND pad, two
between C9 and U1, and a sparse grid. The +24V and +3V3 tracks split
the top pour into regions joined by thin necks; the vias tie each
region to the bottom pour. They stay clear of the unrouted connections
and the mounting-hole keepout, and no drill lands on silkscreen.

C6 pad 2 had a single thermal spoke. A 0.5 mm track now joins it to a
GND via. C7's reference moves right to clear that via.

Co-Authored-By: Claude Opus 5.5 <noreply@anthropic.com>
Routing:
- net GND: track 0.00 -> 1.22 mm, vias 0 -> 32
